Commit message: slightly different PID values and change in mbes position

File: lolo_description/urdf/lolo_auv.urdf.xacro (robot description, xacro)
@@ -174,5 +174,5 @@
   </joint>
   <joint name="$(arg robot_namespace)/mbes_joint" type="fixed">
-    <origin xyz="2.523 0.0155 -0.302" rpy="3.14159 1.53589 0" />
+    <origin xyz="-.751 -0.0155 0.084" rpy="3.14159 1.53589 0" />
     <parent link="$(arg robot_namespace)/base_link"/>
     <child link="$(arg robot_namespace)/mbes_link"/>
